File: merged_lights.kicad_sch (KiCad schematic)
At the start: 62 parts, among them J1 Conn_01x08, J2 Conn_01x08, J3 AVR-ISP-6, J4 Conn_01x02, J5 Conn_01x02, J6 Conn_01x02, J7 Conn_01x08, J8 Conn_01x02, J9 Conn_01x08, Q1 AO3400A, Q2 AO3400A, Q3 AO3400A, Q4 AO3400A, Q5 AO3400A, Q6 AO3400A, Q7 AO3400A, Q8 AO3400A, SW1 SW_Push, U1 ATmega328P-A, U2 ADXL345BCCZ

Commit message: Update merged_lights.kicad_sch
Parts:
- removed C10, C13, C14, C15, C3, C4, C6, C7: C, Capacitor_SMD:C_0805_2012Metric_Pad1.18x1.45mm_HandSolder, symbol Device:C
- added H1, H2, H3, H4: MountingHole_Pad, MountingHole:MountingHole_2.5mm_Pad_Via, symbol Mechanical:MountingHole_Pad
- added H10, H11, H12, H5, H6, H7, H8, H9: MountingHole_Pad, MountingHole:MountingHole_2.5mm_Pad, symbol Mechanical:MountingHole_Pad
- renumbered D2 to D1, D6 to D10, D3 to D2, D1 to D3, D8 to D5, D9 to D6, D10 to D7, D7 to D8, D5 to D9, Q2 to Q1, Q3 to Q2, Q4 to Q3, Q1 to Q4, Q8 to Q7, Q7 to Q8, R4 to R1, R11 to R10, R12 to R11, R13 to R12, R14 to R13, R15 to R14, R17 to R15, R9 to R17, R1 to R2, R2 to R3, R3 to R4, R6 to R5, R7 to R6, R8 to R7, R5 to R8, R10 to R9
Connections:
- net GND: now also H1.1, H2.1, H3.1, H4.1
- no-connect marks 13 -> 21
Other:
- moved on the sheet: Q1, Q2, Q3, Q4, R1, R2, R3, R4, R5, R6, R7, R8
